File: ssd-ps-33.kicad_sch (KiCad schematic)
At the start: 19 parts, among them J1 Top, J2 Bottom, U1 TPS563252

Commit message: Complete BOM with market available parts
Parts:
- D1: Manufacturer (none) -> onsemi; Part Number (none) -> MM3Z5V6ST1G
- J1, J2: Manufacturer (none) -> Adam Tech; Part Number (none) -> PH1-07-UA
- R1: Manufacturer (none) -> YAGEO; Part Number (none) -> RC0603FR-0751KL
- R2: Manufacturer (none) -> YAGEO; Part Number (none) -> RC0603FR-0727KL
- R3: Manufacturer (none) -> YAGEO; Part Number (none) -> RC0603JR-0751RL
- R4: value 135k -> 120k; Manufacturer (none) -> YAGEO; Part Number (none) -> RC0603FR-07120KL
- R5: value 30k -> 26.7k; Manufacturer (none) -> YAGEO; Part Number (none) -> RC0603FR-0726K7L
- R6: Manufacturer (none) -> YAGEO; Part Number (none) -> RC0603FR-0710KL
Other:
- note added: "Vout = 0.6V * (1 + 120k/26.7k) = 3.3V"
- note removed: "Vout = 0.6V * (1 + 135k/30k) = 3.3V"
Changed lines of the file:
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@@
 		(rev "1")
 	)
-	(text "Vout = 0.6V * (1 + 135k/30k) = 3.3V"
+	(text "Vout = 0.6V * (1 + 120k/26.7k) = 3.3V"
 		(exclude_from_sim no)
 		(at 215.9 116.84 0)
@@
 			)
 		)
-		(property "Datasheet" "~"
+		(property "Datasheet" "https://yageogroup.com/content/datasheet/asset/file/PYU-RC_GROUP_51_ROHS_L"
 			(at 101.6 116.84 0)
 			(effects
@@
 			)
 		)
-		(property "Manufacturer" ""
+		(property "Manufacturer" "YAGEO"
 			(at 101.6 116.84 0)
 			(effects
@@
 			)
 		)
-		(property "Part Number" ""
+		(property "Part Number" "RC0603FR-0727KL"
 			(at 101.6 116.84 0)
 			(effects
@@
 			)
 		)
-		(property "Description" "3A Synchronous Buck Converter, Adjustable Output Voltage, 3-17V Input Voltage, 0.6-10V Output Voltage, SOT-563"
+		(property "Description" "3A Synchronous Buck Converter, Adjustable Output Voltage, 3-17V Input, 0.6-10V Output"
 			(at 146.05 91.44 0)
 			(effects
@@
 			)
 		)
-		(property "Datasheet" "~"
+		(property "Datasheet" "https://yageogroup.com/content/datasheet/asset/file/PYU-RC_GROUP_51_ROHS_L"
 			(at 203.2 104.14 0)
 			(effects
@@
 			)
 		)
-		(property "Description" "5%, 0.1 W, AEC-Q200 Grade 0"
+		(property "Description" "5%, 0.1 W"
 			(at 203.2 104.14 0)
 			(effects
@@
 			)
 		)
-		(property "Manufacturer" ""
+		(property "Manufacturer" "YAGEO"
 			(at 203.2 104.14 0)
 			(effects
@@
 			)
 		)
-		(property "Part Number" ""
+		(property "Part Number" "RC0603JR-0751RL"
 			(at 203.2 104.14 0)
 			(effects
@@
 			)
 		)
-		(property "Datasheet" "~"
+		(property "Datasheet" "https://yageogroup.com/content/datasheet/asset/file/PYU-RC_GROUP_51_ROHS_L"
 			(at 101.6 104.14 0)
 			(effects
@@
 			)
 		)
-		(property "Manufacturer" ""
+		(property "Manufacturer" "YAGEO"
 			(at 101.6 104.14 0)
 			(effects
@@
 			)
 		)
-		(property "Part Number" ""
+		(property "Part Number" "RC0603FR-0751KL"
 			(at 101.6 104.14 0)
 			(effects
@@
 			)
 		)
-		(property "Datasheet" "~"
+		(property "Datasheet" "https://yageogroup.com/content/datasheet/asset/file/PYU-RC_GROUP_51_ROHS_L"
 			(at 171.45 85.09 0)
 			(effects
@@
 			)
 		)
-		(property "Description" "1%, 0.1 W, AEC-Q200 Grade 0"
+		(property "Description" "1%, 0.1 W"
 			(at 171.45 85.09 0)
 			(effects
@@
 			)
 		)
-		(property "Manufacturer" ""
+		(property "Manufacturer" "YAGEO"
 			(at 171.45 85.09 0)
 			(effects
@@
 			)
 		)
-		(property "Part Number" ""
+		(property "Part Number" "RC0603FR-0710KL"
 			(at 171.45 85.09 0)
 			(effects
@@
 			)
 		)
-		(property "Datasheet" "~"
+		(property "Datasheet" "https://www.onsemi.com/pdf/datasheet/mm3z2v4st1-d.pdf"
 			(at 88.9 116.84 0)
 			(effects
@@
 			)
 		)
-		(property "Description" "Zener"
+		(property "Description" "Zener, 300mW, ±2%"
 			(at 88.9 116.84 0)
 			(effects
@@
 			)
 		)
-		(property "Manufacturer" ""
+		(property "Manufacturer" "onsemi"
 			(at 88.9 116.84 90)
 			(effects
@@
 			)
 		)
-		(property "Part Number" ""
+		(property "Part Number" "MM3Z5V6ST1G"
 			(at 88.9 116.84 90)
 			(effects
@@
 			)
 		)
-		(property "Value" "135k"
+		(property "Value" "120k"
 			(at 205.74 118.1099 0)
 			(effects
@@
 			)
 		)
-		(property "Datasheet" "~"
+		(property "Datasheet" "https://yageogroup.com/content/datasheet/asset/file/PYU-RC_GROUP_51_ROHS_L"
 			(at 203.2 116.84 0)
 			(effects
@@
 			)
 		)
-		(property "Manufacturer" ""
+		(property "Manufacturer" "YAGEO"
 			(at 203.2 116.84 0)
 			(effects
@@
 			)
 		)
-		(property "Part Number" ""
+		(property "Part Number" "RC0603FR-07120KL"
 			(at 203.2 116.84 0)
 			(effects
@@
 			)
 		)
-		(property "Value" "30k"
+		(property "Value" "26.7k"
 			(at 205.74 130.8099 0)
 			(effects
@@
 			)
 		)
-		(property "Datasheet" "~"
+		(property "Datasheet" "https://yageogroup.com/content/datasheet/asset/file/PYU-RC_GROUP_51_ROHS_L"
 			(at 203.2 129.54 0)
 			(effects
@@
 			)
 		)
-		(property "Description" "1%, 0.1 W, AEC-Q200 Grade 0"
+		(property "Description" "1%, 0.1 W"
 			(at 203.2 129.54 0)
 			(effects
@@
 			)
 		)
-		(property "Manufacturer" ""
+		(property "Manufacturer" "YAGEO"
 			(at 203.2 129.54 0)
 			(effects
@@
 			)
 		)
-		(property "Part Number" ""
+		(property "Part Number" "RC0603FR-0726K7L"
 			(at 203.2 129.54 0)
 			(effects
@@
 			)
 		)
-		(property "Datasheet" "~"
+		(property "Datasheet" "https://app.adam-tech.com/products/download/data_sheet/201605/ph1-xx-ua-data-sheet.pdf"
+			(at 54.61 113.03 0)
+			(effects
+				(font
+					(size 1.27 1.27)
+				)
+				(hide yes)
+			)
+		)
+		(property "Description" "Contact mating 0.236\" (6.00mm), post 0.120\" (3.05mm), insulation 0.098\" (2.50mm)"
 			(at 54.61 113.03 0)
 			(effects
@@
 			)
 		)
-		(property "Description" "Generic connector, single row, 01x07, script generated"
+		(property "Manufacturer" "Adam Tech"
+			(at 54.61 113.03 0)
+			(effects
+				(font
+					(size 1.27 1.27)
+				)
+				(hide yes)
+			)
+		)
+		(property "Part Number" "PH1-07-UA"
 			(at 54.61 113.03 0)
 			(effects
@@
 			)
 		)
-		(property "Datasheet" "~"
+		(property "Datasheet" "https://app.adam-tech.com/products/download/data_sheet/201605/ph1-xx-ua-data-sheet.pdf"
+			(at 54.61 67.31 0)
+			(effects
+				(font
+					(size 1.27 1.27)
+				)
+				(hide yes)
+			)
+		)
+		(property "Description" "Contact mating 0.236\" (6.00mm), post 0.120\" (3.05mm), insulation 0.098\" (2.50mm)"
+			(at 54.61 67.31 0)
+			(effects
+				(font
+					(size 1.27 1.27)
+				)
+				(hide yes)
+			)
+		)
+		(property "Manufacturer" "Adam Tech"
 			(at 54.61 67.31 0)
 			(effects
@@
 			)
 		)
-		(property "Description" "Generic connector, single row, 01x07, script generated"
+		(property "Part Number" "PH1-07-UA"
 			(at 54.61 67.31 0)
 			(effects
